Commit message: refactor: decouple simulation backend from ros2_control macros
Backport from the jazzy branch for PRCUN-6156.

The franka_hardware ros2_control macros (franka_arm and tmrv0_2) used
xacro:if toggles to pick the simulation backend. Decouple them: the
hardware <plugin> block and the gz_ros2_control <gazebo> system element
are now injected by the owning package (franka_bringup for real/mock,
franka_gazebo_bringup for gazebo) rather than selected inside
franka_hardware.

Changes:
- franka_hardware: drop the gazebo/gazebo_effort toggles; expose
  mode/interface selection via capability flags
  (include_effort_command, include_finger_joint, include_passive_base)
- franka_bringup: inject the real/mock hardware plugin from the
  entry-point URDF; relocate the effort-gating test to expand the
  gazebo wrapper
- franka_gazebo_bringup: inject the gz_ros2_control <gazebo> system
  element; collapse five duplicate top-level /**: keys in
  franka_gazebo_controllers.yaml into one — YAML last-key-wins was
  silently dropping the controller_manager type declarations and
  blocking the tmr gazebo launch

URDF expansions remain behavior-equivalent.

File: franka_bringup/urdf/franka_arm.urdf.xacro (robot description, xacro)
@@ -16,5 +16,4 @@
   <xacro:arg name="use_fake_hardware" default="false"/>
   <xacro:arg name="fake_sensor_commands" default="false"/>
-  <xacro:arg name="gazebo_effort" default="false"/>
   <xacro:arg name="is_async" default="false"/>
   <xacro:arg name="thread_priority" default="50"/>
@@ -22,12 +21,22 @@
   <xacro:franka_arm_ros2_control
       robot_type="$(arg robot_type)"
-      robot_ip="$(arg robot_ip)"
-      use_fake_hardware="$(arg use_fake_hardware)"
-      fake_sensor_commands="$(arg fake_sensor_commands)"
-      gazebo="$(arg gazebo)"
-      hand="$(arg hand)"
-      gazebo_effort="$(arg gazebo_effort)"
+      include_effort_command="true"
+      include_finger_joint="false"
       arm_prefix="${modified_prefix}"
       is_async="$(arg is_async)"
-      thread_priority="$(arg thread_priority)"/>
+      thread_priority="$(arg thread_priority)">
+    <hardware_plugin>
+      <!-- Real-vs-mock selection stays at the bringup entry level. -->
+      <xacro:if value="$(arg use_fake_hardware)">
+        <plugin>mock_components/GenericSystem</plugin>
+        <param name="mock_sensor_commands">$(arg fake_sensor_commands)</param>
+        <param name="state_following_offset">0.0</param>
+      </xacro:if>
+      <xacro:unless value="$(arg use_fake_hardware)">
+        <plugin>franka_hardware/FrankaHardwareInterface</plugin>
+        <param name="robot_ip">$(arg robot_ip)</param>
+        <param name="arm_prefix">${modified_prefix}</param>
+      </xacro:unless>
+    </hardware_plugin>
+  </xacro:franka_arm_ros2_control>
 </robot>

File: franka_bringup/urdf/tmrv0_2.urdf.xacro (robot description, xacro)
@@ -22,10 +22,20 @@
   <xacro:tmrv0_2_ros2_control
       mobile_robot_type="tmrv0_2"
-      robot_ip="$(arg robot_ip)"
-      use_fake_hardware="$(arg use_fake_hardware)"
-      fake_sensor_commands="$(arg fake_sensor_commands)"
-      gazebo="false"
-      robot_namespace=""
+      include_passive_base="false"
       is_async="$(arg is_async)"
-      thread_priority="$(arg thread_priority)"/>
+      thread_priority="$(arg thread_priority)">
+    <hardware_plugin>
+      <!-- Real-vs-mock selection stays at the bringup entry level. -->
+      <xacro:if value="$(arg use_fake_hardware)">
+        <plugin>mock_components/GenericSystem</plugin>
+        <param name="mock_gpio_commands">true</param>
+        <param name="mock_sensor_commands">$(arg fake_sensor_commands)</param>
+        <param name="state_following_offset">0.0</param>
+      </xacro:if>
+      <xacro:unless value="$(arg use_fake_hardware)">
+        <plugin>franka_hardware/FrankaHardwareInterface</plugin>
+        <param name="robot_ip">$(arg robot_ip)</param>
+      </xacro:unless>
+    </hardware_plugin>
+  </xacro:tmrv0_2_ros2_control>
 </robot>

File: franka_gazebo/franka_gazebo_bringup/urdf/franka_arm.gazebo.xacro (robot description, xacro)
@@ -31,8 +31,24 @@
     <xacro:franka_arm_ros2_control
         robot_type="$(arg robot_type)"
-        gazebo="true"
-        hand="$(arg hand)"
-        gazebo_effort="$(arg gazebo_effort)"
-        arm_prefix="${modified_prefix}"/>
+        include_effort_command="$(arg gazebo_effort)"
+        include_finger_joint="$(arg hand)"
+        arm_prefix="${modified_prefix}">
+      <hardware_plugin>
+        <!-- Default gz_ros2_control system handles position/velocity; under gazebo_effort
+             the gravity-compensation system is used so effort joints stay compensated. -->
+        <xacro:if value="$(arg gazebo_effort)">
+          <plugin>franka_gazebo_hardware/GazeboGravityCompensationSystem</plugin>
+        </xacro:if>
+        <xacro:unless value="$(arg gazebo_effort)">
+          <plugin>gz_ros2_control/GazeboSimSystem</plugin>
+        </xacro:unless>
+      </hardware_plugin>
+    </xacro:franka_arm_ros2_control>
+    <!-- gz_ros2_control system element (sibling of ros2_control) -->
+    <gazebo>
+      <plugin filename="gz_ros2_control-system" name="gz_ros2_control::GazeboSimROS2ControlPlugin">
+        <parameters>$(find franka_gazebo_bringup)/config/franka_gazebo_controllers.yaml</parameters>
+      </plugin>
+    </gazebo>
     <!-- ================================================================ -->
     <!-- Gazebo sensors                                                    -->

File: franka_gazebo/franka_gazebo_bringup/urdf/tmrv0_2.gazebo.urdf.xacro (robot description, xacro)
@@ -2,26 +2,18 @@
 <!--
   Gazebo entry point for the TMR v0.2 mobile base (without arms).
-  Includes the franka_description base robot and applies ros2_control
-  hardware interface for gazebo simulation.
+  Includes the franka_description robot entry point and applies the
+  ros2_control hardware interface for gazebo simulation.
 -->
 <robot xmlns:xacro="http://www.ros.org/wiki/xacro" name="tmrv0_2_gazebo">
+  <!-- Spawn the base robot in gazebo mode. Declared before the description
+       include so it overrides the entry point's default (false); CLI -D wins. -->
+  <xacro:arg name="gazebo" default="true"/>
   <!-- ================================================================ -->
   <!-- Macro includes                                                    -->
   <!-- ================================================================ -->
-  <xacro:include filename="$(find franka_description)/robots/tmrv0_2/tmrv0_2.xacro"/>
+  <!-- Base robot: reuses the description entry point (declares robot_type,
+       reduced_version, robot_namespace, gazebo and instantiates the robot). -->
+  <xacro:include filename="$(find franka_description)/robots/tmrv0_2/tmrv0_2.urdf.xacro"/>
   <xacro:include filename="$(find franka_hardware)/ros2_control/tmrv0_2.ros2_control.xacro"/>
-  <!-- ================================================================ -->
-  <!-- Arguments                                                        -->
-  <!-- ================================================================ -->
-  <xacro:arg name="robot_type" default="tmrv0_2"/>
-  <xacro:arg name="reduced_version" default="false"/>
-  <xacro:arg name="robot_namespace" default=""/>
-  <!-- ================================================================ -->
-  <!-- Base robot (geometry only)                                       -->
-  <!-- ================================================================ -->
-  <xacro:tmrv0_2 mobile_robot_type="$(arg robot_type)"
-    reduced_version="$(arg reduced_version)"
-    robot_namespace="$(arg robot_namespace)"
-    gazebo="true"/>
   <!-- ================================================================ -->
   <!-- ros2_control hardware interface (gazebo mode)                    -->
@@ -29,5 +21,14 @@
   <xacro:tmrv0_2_ros2_control
     mobile_robot_type="$(arg robot_type)"
-    gazebo="true"
-    robot_namespace="$(arg robot_namespace)"/>
+    include_passive_base="true">
+    <hardware_plugin>
+      <plugin>gz_ros2_control/GazeboSimSystem</plugin>
+    </hardware_plugin>
+  </xacro:tmrv0_2_ros2_control>
+  <!-- gz_ros2_control system element (sibling of ros2_control) -->
+  <gazebo>
+    <plugin filename="gz_ros2_control-system" name="gz_ros2_control::GazeboSimROS2ControlPlugin">
+      <parameters>$(find franka_gazebo_bringup)/config/franka_gazebo_controllers.yaml</parameters>
+    </plugin>
+  </gazebo>
 </robot>

File: franka_gazebo/franka_gazebo_bringup/urdf/tmrv0_2_with_sensors.gazebo.urdf.xacro (robot description, xacro)
@@ -27,5 +27,4 @@
     robot_type="$(arg robot_type)"
     reduced_version="false"
-    gazebo="true"
     robot_namespace="$(arg robot_namespace)"/>
   <!-- ================================================================ -->
@@ -34,6 +33,15 @@
   <xacro:tmrv0_2_ros2_control
     mobile_robot_type="$(arg robot_type)"
-    gazebo="true"
-    robot_namespace="$(arg robot_namespace)"/>
+    include_passive_base="true">
+    <hardware_plugin>
+      <plugin>gz_ros2_control/GazeboSimSystem</plugin>
+    </hardware_plugin>
+  </xacro:tmrv0_2_ros2_control>
+  <!-- gz_ros2_control system element (sibling of ros2_control) -->
+  <gazebo>
+    <plugin filename="gz_ros2_control-system" name="gz_ros2_control::GazeboSimROS2ControlPlugin">
+      <parameters>$(find franka_gazebo_bringup)/config/franka_gazebo_controllers.yaml</parameters>
+    </plugin>
+  </gazebo>
   <!-- ================= CAMERA SENSORS ================= -->
   <xacro:franka_gazebo_camera link_reference="camera_front_link"

File: franka_hardware/ros2_control/franka_ros2_control_macros.xacro (robot description, xacro)
@@ -2,9 +2,9 @@
 <robot xmlns:xacro="http://www.ros.org/wiki/xacro">
   <!-- Configure a single Franka arm joint with position/velocity/conditional-effort commands -->
-  <xacro:macro name="configure_arm_joint" params="joint_name initial_position gazebo:=0 gazebo_effort:=0">
+  <xacro:macro name="configure_arm_joint" params="joint_name initial_position include_effort_command:=1">
     <joint name="${joint_name}">
       <command_interface name="position"/>
       <command_interface name="velocity"/>
-      <xacro:if value="${gazebo == 0 or gazebo_effort == 1}">
+      <xacro:if value="${include_effort_command}">
         <command_interface name="effort"/>
       </xacro:if>
@@ -17,20 +17,20 @@
   </xacro:macro>
   <!-- Configure all 7 arm joints for a given prefix with standard initial positions -->
-  <xacro:macro name="configure_arm_joints" params="joint_prefix gazebo:=0 gazebo_effort:=0">
-    <xacro:configure_arm_joint joint_name="${joint_prefix}_joint1" initial_position="0.0" gazebo="${gazebo}" gazebo_effort="${gazebo_effort}"/>
-    <xacro:configure_arm_joint joint_name="${joint_prefix}_joint2" initial_position="${-pi/4}" gazebo="${gazebo}" gazebo_effort="${gazebo_effort}"/>
-    <xacro:configure_arm_joint joint_name="${joint_prefix}_joint3" initial_position="0.0" gazebo="${gazebo}" gazebo_effort="${gazebo_effort}"/>
-    <xacro:configure_arm_joint joint_name="${joint_prefix}_joint4" initial_position="${-3*pi/4}" gazebo="${gazebo}" gazebo_effort="${gazebo_effort}"/>
-    <xacro:configure_arm_joint joint_name="${joint_prefix}_joint5" initial_position="0.0" gazebo="${gazebo}" gazebo_effort="${gazebo_effort}"/>
-    <xacro:configure_arm_joint joint_name="${joint_prefix}_joint6" initial_position="${pi/2}" gazebo="${gazebo}" gazebo_effort="${gazebo_effort}"/>
-    <xacro:configure_arm_joint joint_name="${joint_prefix}_joint7" initial_position="${pi/4}" gazebo="${gazebo}" gazebo_effort="${gazebo_effort}"/>
+  <xacro:macro name="configure_arm_joints" params="joint_prefix include_effort_command:=1">
+    <xacro:configure_arm_joint joint_name="${joint_prefix}_joint1" initial_position="0.0" include_effort_command="${include_effort_command}"/>
+    <xacro:configure_arm_joint joint_name="${joint_prefix}_joint2" initial_position="${-pi/4}" include_effort_command="${include_effort_command}"/>
+    <xacro:configure_arm_joint joint_name="${joint_prefix}_joint3" initial_position="0.0" include_effort_command="${include_effort_command}"/>
+    <xacro:configure_arm_joint joint_name="${joint_prefix}_joint4" initial_position="${-3*pi/4}" include_effort_command="${include_effort_command}"/>
+    <xacro:configure_arm_joint joint_name="${joint_prefix}_joint5" initial_position="0.0" include_effort_command="${include_effort_command}"/>
+    <xacro:configure_arm_joint joint_name="${joint_prefix}_joint6" initial_position="${pi/2}" include_effort_command="${include_effort_command}"/>
+    <xacro:configure_arm_joint joint_name="${joint_prefix}_joint7" initial_position="${pi/4}" include_effort_command="${include_effort_command}"/>
   </xacro:macro>
   <!-- Configure a finger joint (position_only=1 omits velocity/effort commands) -->
-  <xacro:macro name="configure_finger_joint" params="joint_name gazebo:=0 gazebo_effort:=0 position_only:=0">
+  <xacro:macro name="configure_finger_joint" params="joint_name include_effort_command:=1 position_only:=0">
     <joint name="${joint_name}">
       <command_interface name="position"/>
       <xacro:unless value="${position_only}">
         <command_interface name="velocity"/>
-        <xacro:if value="${gazebo == 0 or gazebo_effort == 1}">
+        <xacro:if value="${include_effort_command}">
           <command_interface name="effort"/>
         </xacro:if>
@@ -86,11 +86,11 @@
   </xacro:macro>
   <!-- Emit 6 cartesian_velocity GPIO entries (vx, vy, vz, wx, wy, wz) for a given prefix -->
-  <xacro:macro name="cartesian_velocity_io" params="prefix:='' start_index:=0">
-    <xacro:general_purpose_io prefix="${prefix}vx" command_interface="cartesian_velocity" index="${start_index + 0}"/>
-    <xacro:general_purpose_io prefix="${prefix}vy" command_interface="cartesian_velocity" index="${start_index + 1}"/>
-    <xacro:general_purpose_io prefix="${prefix}vz" command_interface="cartesian_velocity" index="${start_index + 2}"/>
-    <xacro:general_purpose_io prefix="${prefix}wx" command_interface="cartesian_velocity" index="${start_index + 3}"/>
-    <xacro:general_purpose_io prefix="${prefix}wy" command_interface="cartesian_velocity" index="${start_index + 4}"/>
-    <xacro:general_purpose_io prefix="${prefix}wz" command_interface="cartesian_velocity" index="${start_index + 5}"/>
+  <xacro:macro name="cartesian_velocity_io" params="prefix:=''">
+    <xacro:general_purpose_io prefix="${prefix}vx" command_interface="cartesian_velocity" index="0"/>
+    <xacro:general_purpose_io prefix="${prefix}vy" command_interface="cartesian_velocity" index="1"/>
+    <xacro:general_purpose_io prefix="${prefix}vz" command_interface="cartesian_velocity" index="2"/>
+    <xacro:general_purpose_io prefix="${prefix}wx" command_interface="cartesian_velocity" index="3"/>
+    <xacro:general_purpose_io prefix="${prefix}wy" command_interface="cartesian_velocity" index="4"/>
+    <xacro:general_purpose_io prefix="${prefix}wz" command_interface="cartesian_velocity" index="5"/>
   </xacro:macro>
   <!-- Configure the 4 TMR drive joints (2 steering + 2 driving) -->
@@ -124,24 +124,23 @@
   </xacro:macro>
   <!-- Complete per-arm interface set: joints + finger + cartesian_velocity + elbow + cartesian_pose + sensor.
-       Each component is optional via boolean flags. Indices are parameterized for shared hardware blocks. -->
+       Each component is optional via boolean flags. Indices start at 0 (single-arm hardware block). -->
   <xacro:macro name="configure_arm_interfaces"
-    params="joint_prefix gpio_prefix gazebo:=0 gazebo_effort:=0 hand:=0
-            cv_start_index:=0
-            include_elbow:=0 elbow_start_index:=0
+    params="joint_prefix gpio_prefix include_effort_command:=1 include_finger_joint:=0
+            include_elbow:=0
             include_cartesian_pose:=0
             include_sensor:=0 sensor_name:=''
             finger_position_only:=0">
     <!-- 7 arm joints (position/velocity/conditional-effort) -->
-    <xacro:configure_arm_joints joint_prefix="${joint_prefix}" gazebo="${gazebo}" gazebo_effort="${gazebo_effort}"/>
-    <!-- Finger joint (only in gazebo with hand) -->
-    <xacro:if value="${gazebo and hand}">
-      <xacro:configure_finger_joint joint_name="${joint_prefix}_finger_joint1" gazebo="${gazebo}" gazebo_effort="${gazebo_effort}" position_only="${finger_position_only}"/>
+    <xacro:configure_arm_joints joint_prefix="${joint_prefix}" include_effort_command="${include_effort_command}"/>
+    <!-- Optional finger joint -->
+    <xacro:if value="${include_finger_joint}">
+      <xacro:configure_finger_joint joint_name="${joint_prefix}_finger_joint1" include_effort_command="${include_effort_command}" position_only="${finger_position_only}"/>
     </xacro:if>
     <!-- Cartesian velocity GPIOs (6 entries: vx–wz) -->
-    <xacro:cartesian_velocity_io prefix="${gpio_prefix}" start_index="${cv_start_index}"/>
+    <xacro:cartesian_velocity_io prefix="${gpio_prefix}"/>
     <!-- Elbow command GPIOs (2 entries: joint_3_position, joint_4_sign) -->
     <xacro:if value="${include_elbow}">
-      <xacro:general_purpose_io prefix="${gpio_prefix}joint_3_position" command_interface="elbow_command" index="${elbow_start_index + 0}"/>
-      <xacro:general_purpose_io prefix="${gpio_prefix}joint_4_sign" command_interface="elbow_command" index="${elbow_start_index + 1}"/>
+      <xacro:general_purpose_io prefix="${gpio_prefix}joint_3_position" command_interface="elbow_command" index="0"/>
+      <xacro:general_purpose_io prefix="${gpio_prefix}joint_4_sign" command_interface="elbow_command" index="1"/>
     </xacro:if>
     <!-- Cartesian pose GPIOs (16 entries) -->

File: franka_mobile_sensors/robots/tmrv0_2_with_sensors.urdf.xacro (robot description, xacro)
@@ -6,20 +6,16 @@
   <!-- Should the reduced kinematic version (without caster wheels) be used? -->
   <xacro:arg name="reduced_version" default="false" />
-  <!-- Should the robot be spawned in Gazebo? -->
-  <xacro:arg name="gazebo" default="false" />
   <!-- The namespace of the robot -->
   <xacro:arg name="robot_namespace" default="" />
-  <xacro:unless value="$(arg gazebo)">
-    <link name="base"/>
-    <joint name="base_joint" type="fixed">
-      <parent link="base"/>
-      <child link="base_link"/>
-      <origin rpy="0 0 0" xyz="0 0 0"/>
-    </joint>
-  </xacro:unless>
+  <!-- Fixed root link for the standalone (non-simulation) robot description. -->
+  <link name="base"/>
+  <joint name="base_joint" type="fixed">
+    <parent link="base"/>
+    <child link="base_link"/>
+    <origin rpy="0 0 0" xyz="0 0 0"/>
+  </joint>
   <xacro:tmrv0_2_with_sensors
             robot_type="$(arg robot_type)"
             reduced_version="$(arg reduced_version)"
-            robot_namespace="$(arg robot_namespace)"
-            gazebo="$(arg gazebo)"/>
+            robot_namespace="$(arg robot_namespace)"/>
 </robot>

File: franka_mobile_sensors/robots/tmrv0_2_with_sensors.xacro (robot description, xacro)
@@ -12,11 +12,9 @@
       params="robot_type
               reduced_version
-              gazebo
               robot_namespace">
     <!-- Instantiate the base robot (Layer 1) -->
     <xacro:tmrv0_2 mobile_robot_type="${robot_type}"
                 reduced_version="${reduced_version}"
-                robot_namespace="${robot_namespace}"
-                gazebo="${gazebo}"/>
+                robot_namespace="${robot_namespace}"/>
     <!-- Attach all sensors -->
     <xacro:sensor_suite />
