Commit message: fix: correctly pick up meshes for nanoscan lidar

File: franka_mobile_sensors/robots/nanoscan3/nanoscan3/nanoscan3_macro.xacro (robot description, xacro)
@@ -33,5 +33,5 @@
         <visual>
           <geometry>
-            <mesh filename="file://$(find sick_safetyscanners2)/meshes/nanoscan3/MountingKit_2a.dae"/>
+            <mesh filename="package://sick_safetyscanners2/description/meshes/MountingKit_2a.dae"/>
           </geometry>
           <material name="black">
@@ -41,5 +41,5 @@
         <collision>
           <geometry>
-            <mesh filename="file://$(find sick_safetyscanners2)/meshes/nanoscan3/MountingKit_2a_collision.stl"/>
+            <mesh filename="package://sick_safetyscanners2/description/meshes/MountingKit_2a_collision.stl"/>
           </geometry>
         </collision>
@@ -74,5 +74,5 @@
         <origin xyz="-0.01 -0.08 ${-sensor_z}" rpy="0 0 1.57" />
         <geometry>
-          <mesh filename="file://$(find sick_safetyscanners2)/description/meshes/NANS3.dae"/>
+          <mesh filename="package://sick_safetyscanners2/description/meshes/NANS3.dae"/>
         </geometry>
         <material name="black">
@@ -84,5 +84,5 @@
         <origin xyz="-0.01 -0.08 ${-sensor_z}" rpy="0 0 1.57" />
         <geometry>
-          <mesh filename="file://$(find sick_safetyscanners2)/description/meshes/NANS3_collision.stl"/>
+          <mesh filename="package://sick_safetyscanners2/description/meshes/NANS3_collision.stl"/>
         </geometry>
       </collision>
