Commit message: feat(franka_description_extensions): relocate mobile sensors and vision kit under umbrella package
- Move franka_mobile_sensors and franka_vision_and_manipulation_kit under
  franka_description_extensions/ without changing their ROS package identities
- Repair standalone Layer-2 xacro composition after Gazebo decoupling: drop the
  stale `gazebo` arg, always emit the base link/joint, thread
  `include_self_collision_geometry` through to Layer 1, and expose arm-extras
  hooks on mobile_fr3_duo_v0_2_with_sensors
- Add the umbrella guide (composition layers, mounting points, custom grippers,
  naming/prefixes, examples, troubleshooting) under
  `franka_description_extensions/doc/` (matching the sibling packages' `doc/`
  layout), wire franka_description_extensions into the root docs toctree in
  place of the old per-package entries, and record the change in CHANGELOG.rst
- Add package-owned installed-share xacro expansion and graph-validity
  regression tests for both packages, with the CMake/package.xml test
  dependencies they require
- Clean up the reviewed xacro arg comments to be declarative
- Fix both Duo Gazebo launches to preserve and de-duplicate any caller-supplied
  `GZ_SIM_RESOURCE_PATH` instead of overwriting it, and include the
  `realsense2_description` share root so the D405 mesh resolves; declare the
  new direct RealSense/test dependencies in package.xml and add a
  resource-resolution regression test

Validated in the Jazzy container: focused docs and 27 vision xacro tests pass;
clean Gazebo package build/tests pass; 27 affected bringup tests pass;
stationary and mobile headless sensor Gazebo runs report zero
`model://`/D405 errors and were fully torn down; final diff checks clean.

Co-authored-by: Cursor <cursoragent@cursor.com>

File: franka_description_extensions/franka_mobile_sensors/robots/mobile_fr3_duo_v0_2_with_sensors.urdf.xacro (robot description, xacro)
@@ -25,6 +25,6 @@
   <!-- Should self-collision be enabled? -->
   <xacro:arg name="with_sc" default="false" />
-  <!-- Should the robot be spawned in Gazebo? -->
-  <xacro:arg name="gazebo" default="false" />
+  <!-- Emit the coarse self-collision capsule geometry inside the *_sc sub-links? -->
+  <xacro:arg name="include_self_collision_geometry" default="true" />
   <!-- Name of the description package -->
   <xacro:arg name="description_pkg" default="franka_description" />
@@ -35,16 +35,13 @@
   <!-- Should the arms be used? -->
   <xacro:arg name="use_arms" default="true" />
-  <xacro:unless value="$(arg gazebo)">
-    <link name="base"/>
-    <joint name="base_joint" type="fixed">
-      <parent link="base"/>
-      <child link="base_link"/>
-      <origin rpy="0 0 0" xyz="0 0 0"/>
-    </joint>
-  </xacro:unless>
+  <link name="base"/>
+  <joint name="base_joint" type="fixed">
+    <parent link="base"/>
+    <child link="base_link"/>
+    <origin rpy="0 0 0" xyz="0 0 0"/>
+  </joint>
   <xacro:mobile_fr3_duo_v0_2_with_sensors
         robot_types="$(arg robot_types)"
         hand="$(arg hand)"
-        gazebo="$(arg gazebo)"
         reduced_version="$(arg reduced_version)"
         description_pkg="$(arg description_pkg)"
@@ -59,4 +56,5 @@
         tcp_rpy="$(arg tcp_rpy)"
         safety_distance="$(arg safety_distance)"
-        with_sc="$(arg with_sc)"/>
+        with_sc="$(arg with_sc)"
+        include_self_collision_geometry="$(arg include_self_collision_geometry)"/>
 </robot>

File: franka_description_extensions/franka_mobile_sensors/robots/mobile_fr3_duo_v0_2_with_sensors.xacro (robot description, xacro)
@@ -5,8 +5,5 @@
     - Layer 1 macro (franka_description: mobile_fr3_duo_v0_2)
     - Sensor suite  (franka_mobile_sensors: sensor_suite)
-  Callers must define the following properties before invoking this macro
-  (required by the Layer 1 macro):
-    robot_types_list   — Python list, e.g. ${['tmrv0_2','fr3v2','fr3v2']}
-    robot_ips_list     — Python list, e.g. ${['172.16.0.1','172.16.0.2','172.16.0.3']}
+  Callers must define robot_types_list before invoking this macro.
 -->
 <robot xmlns:xacro="http://www.ros.org/wiki/xacro">
@@ -25,5 +22,5 @@
               safety_distance
               with_sc
-              gazebo
+              include_self_collision_geometry
               description_pkg
               connected_to
@@ -34,5 +31,4 @@
           robot_types="${robot_types}"
           hand="${hand}"
-          gazebo="${gazebo}"
           reduced_version="${reduced_version}"
           description_pkg="${description_pkg}"
@@ -47,5 +43,9 @@
           tcp_rpy="${tcp_rpy}"
           safety_distance="${safety_distance}"
-          with_sc="${with_sc}"/>
+          with_sc="${with_sc}"
+          include_self_collision_geometry="${include_self_collision_geometry}">
+      <arm0_extras/>
+      <arm1_extras/>
+    </xacro:mobile_fr3_duo_v0_2>
     <!-- Attach all sensors -->
     <xacro:sensor_suite />

File: franka_description_extensions/franka_mobile_sensors/robots/tmrv0_2_with_sensors.urdf.xacro (robot description, xacro)
@@ -6,20 +6,15 @@
   <!-- Should the reduced kinematic version (without caster wheels) be used? -->
   <xacro:arg name="reduced_version" default="false" />
-  <!-- Should the robot be spawned in Gazebo? -->
-  <xacro:arg name="gazebo" default="false" />
   <!-- The namespace of the robot -->
   <xacro:arg name="robot_namespace" default="" />
-  <xacro:unless value="$(arg gazebo)">
-    <link name="base"/>
-    <joint name="base_joint" type="fixed">
-      <parent link="base"/>
-      <child link="base_link"/>
-      <origin rpy="0 0 0" xyz="0 0 0"/>
-    </joint>
-  </xacro:unless>
+  <link name="base"/>
+  <joint name="base_joint" type="fixed">
+    <parent link="base"/>
+    <child link="base_link"/>
+    <origin rpy="0 0 0" xyz="0 0 0"/>
+  </joint>
   <xacro:tmrv0_2_with_sensors
             robot_type="$(arg robot_type)"
             reduced_version="$(arg reduced_version)"
-            robot_namespace="$(arg robot_namespace)"
-            gazebo="$(arg gazebo)"/>
+            robot_namespace="$(arg robot_namespace)"/>
 </robot>

File: franka_description_extensions/franka_vision_and_manipulation_kit/robots/vision_and_manipulation_kit.urdf.xacro (robot description, xacro)
@@ -24,7 +24,9 @@
   <!-- Safety distance for the collision capsules -->
   <xacro:arg name="safety_distance" default="0.03" />
-  <!-- Should self-collision be enabled? -->
+  <!-- Enable self-collision geometry. -->
   <xacro:arg name="with_sc" default="false" />
-  <!-- Is the robot being controlled with ros2_control?" -->
+  <!-- Emit the coarse self-collision capsule geometry inside the *_sc sub-links? -->
+  <xacro:arg name="include_self_collision_geometry" default="true" />
+  <!-- Is the robot being controlled with ros2_control? -->
   <xacro:arg name="ros2_control" default="false" />
   <!-- IP address or hostname of the robot" -->
@@ -36,8 +38,4 @@
   <!-- Should fake sensors be used? -->
   <xacro:arg name="fake_sensor_commands" default="false" />
-  <!-- Should the robot be spawned in Gazebo?" -->
-  <xacro:arg name="gazebo" default="false" />
-  <!-- Should the robot be spawned in Gazebo with effort interfaces?" -->
-  <xacro:arg name="gazebo_effort" default="false" />
   <!-- Name of the description package -->
   <xacro:arg name="description_pkg" default="franka_description" />
@@ -56,4 +54,5 @@
     safety_distance="$(arg safety_distance)"
     with_sc="$(arg with_sc)"
+    include_self_collision_geometry="$(arg include_self_collision_geometry)"
     ros2_control="$(arg ros2_control)"
     mobile_platform_ip="$(arg mobile_platform_ip)"
@@ -62,6 +61,4 @@
     use_fake_hardware="$(arg use_fake_hardware)"
     fake_sensor_commands="$(arg fake_sensor_commands)"
-    gazebo="$(arg gazebo)"
-    gazebo_effort="$(arg gazebo_effort)"
     description_pkg="$(arg description_pkg)"
   />

File: franka_description_extensions/franka_vision_and_manipulation_kit/robots/vision_kit_components.xacro (robot description, xacro)
@@ -12,10 +12,10 @@
   <xacro:include filename="$(find zed_description)/urdf/zed_macro.urdf.xacro"/>
   <xacro:macro name="vision_kit_components"
-    params="left_arm_type:=fr3v2 right_arm_type:=fr3v2 prefix:='' robotiq_use_fake_hardware:=false robotiq_include_ros2_control:=true sim_gazebo:=false">
+    params="left_arm_type:=fr3v2 right_arm_type:=fr3v2 prefix:='' left_arm_prefix:='left' right_arm_prefix:='right' robotiq_use_fake_hardware:=false robotiq_include_ros2_control:=true sim_gazebo:=false">
     <!-- Robotiq Grippers with RealSense D405 wrist cameras -->
-    <xacro:robotiq_gripper_with_realsense_camera parent="left_${left_arm_type}_link8" prefix="${prefix}left_"
+    <xacro:robotiq_gripper_with_realsense_camera parent="${left_arm_prefix}_${left_arm_type}_link8" prefix="${prefix}left_"
       robotiq_name="left_robotiq_gripper_hardware" robotiq_use_fake_hardware="${robotiq_use_fake_hardware}"
       robotiq_include_ros2_control="${robotiq_include_ros2_control}" robotiq_sim_gazebo="${sim_gazebo}" />
-    <xacro:robotiq_gripper_with_realsense_camera parent="right_${right_arm_type}_link8" prefix="${prefix}right_"
+    <xacro:robotiq_gripper_with_realsense_camera parent="${right_arm_prefix}_${right_arm_type}_link8" prefix="${prefix}right_"
       robotiq_name="right_robotiq_gripper_hardware" robotiq_use_fake_hardware="${robotiq_use_fake_hardware}"
       robotiq_include_ros2_control="${robotiq_include_ros2_control}" robotiq_sim_gazebo="${sim_gazebo}" />
